File: S-Worm_PCB_Designs/S-Worm_PCB_Designs.kicad_sch (KiCad schematic)
At the start: 0 parts

Commit message: bruh
Parts:
- added U?: ICM-45686, easyeda2kicad:LGA-14_L3.0-W2.5-P0.50-TL, symbol easyeda2kicad:ICM-45686
- added U?: STM32G474RBT6, easyeda2kicad:LQFP-64_L10.0-W10.0-P0.50-LS12.0-BL, symbol easyeda2kicad:STM32G474RBT6
- added U?: BMP580, easyeda2kicad:LGA-10_L2.0-W2.0-P0.50-TL_BMP580, symbol easyeda2kicad:BMP580
- added U?: TPS63070RNMR, easyeda2kicad:VQFN-15_L3.0-W2.5-P0.50-BL, symbol easyeda2kicad:TPS63070RNMR
- added USB?: TYPE-C 16PIN 2MD, easyeda2kicad:USB-C-SMD_TYPE-C-16PIN-2MD-073, symbol easyeda2kicad:TYPE-C16PIN2MD

Commit message: req?
Parts:
- removed U?: TPS63070RNMR, easyeda2kicad:VQFN-15_L3.0-W2.5-P0.50-BL, symbol easyeda2kicad:TPS63070RNMR
- added D? (x3): LED, symbol Device:LED
- added U?: SX1276IMLTRT, easyeda2kicad:QFN-28_L6.0-W6.0-P0.65-BL-EP, symbol easyeda2kicad:SX1276IMLTRT
- added U?: TPS62130RGTR, easyeda2kicad:QFN-16_L3.0-W3.0-P0.50-TL-EP1.7, symbol easyeda2kicad:TPS62130RGTR
- added U?: MAX-M10S-00B, easyeda2kicad:SMD-18_L10.1-W9.7-P1.10-TL_SKG09F, symbol easyeda2kicad:MAX-M10S-00B

Commit message: mag
Parts:
- added C?: 10uF, symbol Device:C
- added C?: 0.1uF, symbol Device:C
- added C?: 22uf, symbol Device:C
- added C?: 3.3nF, symbol Device:C
- added L?: 2.2 uH, symbol Device:L
- added R?: 100k, symbol Device:R_US
Connections:
- net B_VIN: now reaches U?.10 (AVIN)
- net B_VIN: now also U?.12 (PVIN), U?.13 (EN), C?.1, C?.1
- net 3.3Vout: now reaches U?.14 (VOS)
- net 3.3Vout: now also C?.1, L?.2, R?.1
- net GND: now reaches U?.15 (PGND)
- net GND: now also U?.5 (FB), U?.6 (AGND), U?.7 (FSW), U?.8 (DEF), C?.2, C?.2, C?.2, C?.2
- net at U?.3 (SW): now also L?.1
- net at U?.4 (PG): now also R?.2
- net at U?.9 (SS/TR): now also C?.1

Commit message: switching the module lol
Parts:
- added C? (x2): 100nF, symbol Device:C
- added C? (x2): C, symbol Device:C
- added C?: 10uF, symbol Device:C_Small
- added J?: Conn_Coaxial, symbol Connector:Conn_Coaxial
- added R?, Rr: 2.7k, symbol Device:R_Small_US
- added U?: MMC5983MA, easyeda2kicad:LGA-16_L3.0-W3.0-P0.50-BL_SQ, symbol easyeda2kicad:MMC5983MA
Connections:
- net 3.3Vout is gone; now on net +3.3V: C?.1, L?.2, R?.1, U?.14 (VOS)
- net GND is gone; now on net +3.3V: C?.2, C?.2, C?.2, C?.2, U?.15 (PGND), U?.5 (FB), U?.6 (AGND), U?.7 (FSW), U?.8 (DEF)
- net ICM_SDO: now reaches U?.1 (AP_SDO/AP_AD0)
- net ICM_CS: now reaches U?.12 (AP_CS)
- net ICM_SCK: now reaches U?.13 (AP_SCL/AP_SCLK)
- net ICM_SDI: now reaches U?.14 (AP_SDA/AP_SDIO/AP_SDI)
- net +3.3V: now reaches U?.4 (INT1/INT)
- net +3.3V: now also U?.1 (GND), U?.1 (VDDIO), U?.10 (VDD), U?.3 (VSS), U?.5 (SDO), U?.5 (VDDIO), U?.6 (CSB), U?.6 (GND), U?.7 (V_IO), U?.8 (VCC), U?.8 (VDD), U?.8 (VSS), U?.9 (VSS), C?.1, C?.1, C?.1, C?.1, C?.2, C?.2, C?.2, C?.2, C?.2, R?.2, Rr.2, U?.11 (GND), U?.13 (VDDIO), U?.2 (VDD), U?.4 (SPI_CS), U?.9 (GND)
- net ICM_INT2: now reaches U?.9 (INT2/FSYNC/CLKIN)
- net at U?.10 (GND): now also J?.2 (Ext)
- net at U?.11 (RF_IN): now also J?.1 (In)
- net STM32_RX: now reaches U?.2 (TXD)
- net STM32_TX: now reaches U?.3 (RXD)
- net I2C_SCL: now reaches U?.2 (SCK)
- net I2C_SDA: now reaches U?.4 (SDI)
- net BMP_INT: now reaches U?.7 (INT)
- new net: R?.1, U?.16 (SDA/SPI_SDI)
- new net: Rr.1, U?.1 (SCL/SPI_SCK)
- new net: C?.1, U?.10 (CAP)
- no-connect marks 0 -> 5
Other:
- moved on the sheet: U?

Commit message: power_aaa
Parts:
- removed U?: SX1276IMLTRT, easyeda2kicad:QFN-28_L6.0-W6.0-P0.65-BL-EP, symbol easyeda2kicad:SX1276IMLTRT
- removed U?: STM32G474RBT6, easyeda2kicad:LQFP-64_L10.0-W10.0-P0.50-LS12.0-BL, symbol easyeda2kicad:STM32G474RBT6
- added C? (x2): 2.2uF, symbol Device:C_Small
- added C?: 10uF, symbol Device:C_Small
- added C? (x7): 100nF, symbol Device:C_Small
- added C? (x3): 1uF, symbol Device:C_Small
- added C? (x2): 6.8pF, symbol Device:C_Small
- added C? (x2): 20pF, symbol Device:C_Small
- added FB?: FerriteBead_Small, symbol Device:FerriteBead_Small
- added J?: Conn_Coaxial, symbol Connector:Conn_Coaxial
- added R?: R_Small_US, symbol Device:R_Small_US
- added SW? (x2): TS-1088-AR02016, easyeda2kicad:SW-SMD_L3.9-W3.0-P4.45, symbol easyeda2kicad:TS-1088-AR02016
- added U? (x2): STM32F405RGT6, easyeda2kicad:LQFP-64_L10.0-W10.0-P0.50-LS12.0-BL, symbol easyeda2kicad:STM32F405RGT6
- added U?: E22-900M22S, easyeda2kicad:WIRELM-SMD_E22-900M22S, symbol easyeda2kicad:E22-900M22S
- added X?: X322525MOB4SI, easyeda2kicad:CRYSTAL-SMD_4P-L3.2-W2.5-BL, symbol easyeda2kicad:X322525MOB4SI
- added X?: Q13FC1350000400, easyeda2kicad:FC-135R_L3.2-W1.5, symbol easyeda2kicad:Q13FC1350000400
Connections:
- net +3.3V: now also C?.1, C?.1, C?.1, C?.1, C?.1, C?.1, C?.1, C?.1, C?.1, C?.1, C?.1, C?.2, C?.2, C?.2, C?.2, C?.2, C?.2, C?.2, C?.2, C?.2, C?.2, C?.2, C?.2, C?.2, C?.2, FB?.1, J?.2 (Ext), R?.2, SW?.1, SW?.1, U?.1 (GND), U?.1 (VBAT), U?.10 (GND), U?.11 (GND), U?.12 (GND), U?.12 (VSSA), U?.18 (VSS), U?.19 (VDD), U?.2 (GND), U?.20 (GND), U?.22 (GND), U?.3 (GND), U?.32 (VDD), U?.4 (GND), U?.48 (VDD), U?.5 (GND), U?.63 (VSS), U?.64 (VDD), U?.9 (VCC), X?.2 (GND), X?.4 (GND)
- new net: C?.1, U?.31 (VCAP_1)
- new net: C?.1, U?.47 (VCAP_2)
- new net: FB?.2, U?.13 (VDDA)
- new net: J?.1 (In), U?.21 (ANT)
- new net BOOT: R?.1, SW?.2
- new net HSE_in: C?.1, X?.1 (OSC1)
- new net HSE_out: C?.1, X?.3 (OSC2)
- new net LSE_in: C?.1, X?.1
- new net LSE_out: C?.1, X?.2
- new net RESET: C?.2, SW?.2
- new net STM32_MISO: U?.16 (MISO)
- new net STM32_MOSI: U?.17 (MOSI)
- new net STM32_NSS: U?.19 (NSS)
- new net STM32_SCK: U?.18 (SCK)
- new net STM32_TELE_BUSY: U?.14 (BUSY)
- new net STM32_TELE_MSG: U?.13 (DIO1)
- new net STM32_TELE_RST: U?.15 (NRST)
Other:
- moved on the sheet: C?, D?, U?, USB?

Commit message: erm
Parts:
- removed R?, Rr: 2.7k, symbol Device:R_Small_US
- removed USB?: TYPE-C 16PIN 2MD, easyeda2kicad:USB-C-SMD_TYPE-C-16PIN-2MD-073, symbol easyeda2kicad:TYPE-C16PIN2MD
- added C?: 1uF, symbol Device:C_Small
- added C?: 100nF, symbol Device:C_Small
- added J?: Conn_01x02_Socket, symbol Connector:Conn_01x02_Socket
- added J?: USB_A, symbol Connector:USB_A
- added R?: 10k, symbol Device:R_Small_US
- added R?: 80k, symbol Device:R_Small_US
- added R?: 75k, symbol Device:R_Small_US
- added U?: TPS2121RUXR, easyeda2kicad:VQFN-HR-12_L2.5-W2.0-P0.50-BL, symbol easyeda2kicad:TPS2121RUXR
Connections:
- net +3.3V: now also C?.1; no longer C?.1, C?.2, C?.2, C?.2, C?.2, C?.2, C?.2, C?.2, C?.2, C?.2, C?.2, C?.2, C?.2, C?.2, C?.2, C?.2, C?.2, C?.2, C?.2, C?.2, C?.2, C?.2, C?.2, C?.2, J?.2 (Ext), R?.2, SW?.1, U?.1 (GND), U?.1 (GND), U?.10 (GND), U?.11 (GND), U?.11 (GND), U?.12 (GND), U?.12 (VSSA), U?.15 (PGND), U?.18 (VSS), U?.2 (GND), U?.20 (GND), U?.22 (GND), U?.3 (GND), U?.3 (VSS), U?.4 (GND), U?.4 (SPI_CS), U?.5 (FB), U?.5 (GND), U?.5 (SDO), U?.6 (AGND), U?.6 (CSB), U?.6 (GND), U?.63 (VSS), U?.7 (FSW), U?.8 (DEF), U?.8 (VSS), U?.9 (GND), U?.9 (VSS), X?.2 (GND), X?.4 (GND)
- net BOOT: now also U?.60 (BOOT0)
- net RESET: now also U?.7 (NRST)
- net M_SDI: now reaches U?.16 (SDA/SPI_SDI)
- net M_SCK: now reaches U?.1 (SCL/SPI_SCK)
- net M_SDO: now reaches U?.5 (SPI_SDO)
- net B_VIN: no longer names the net of C?.1, C?.1, U?.10 (AVIN), U?.12 (PVIN), U?.13 (EN)
- net B_VIN: now also U?.1 (OUT)
- net STM32_MISO renamed TELE_MISO
- net STM32_MOSI renamed TELE_MOSI
- net STM32_NSS renamed TELE_NSS
- net STM32_SCK renamed TELE_SCK
- net STM32_TELE_BUSY renamed TELE_BUSY
- net STM32_TELE_MSG renamed TELE_MSG
- net STM32_TELE_RST renamed TELE_RST
- new net: R?.1, R?.2, U?.6 (PR1)
- new net: R?.1, U?.10 (ILM)
- new net: C?.1, U?.11 (SS)
- new net D+: J?.3 (D+)
- new net D-: J?.2 (D-)
- new net GND: C?.1, C?.2, C?.2, C?.2, C?.2, C?.2, C?.2, C?.2, C?.2, C?.2, C?.2, C?.2, C?.2, C?.2, C?.2, C?.2, C?.2, C?.2, C?.2, C?.2, C?.2, C?.2, C?.2, C?.2, C?.2, C?.2, J?.2 (Ext), J?.2 (Pin_2), J?.4 (GND), J?.5 (Shield), R?.1, R?.2, R?.2, SW?.1, U?.1 (GND), U?.1 (GND), U?.10 (GND), U?.11 (GND), U?.11 (GND), U?.12 (GND), U?.12 (GND), U?.12 (VSSA), U?.15 (PGND), U?.18 (VSS), U?.2 (GND), U?.20 (GND), U?.22 (GND), U?.3 (CP2), U?.3 (GND), U?.3 (VSS), U?.4 (GND), U?.5 (FB), U?.5 (GND), U?.5 (SDO), U?.6 (AGND), U?.6 (CSB), U?.6 (GND), U?.63 (VSS), U?.7 (FSW), U?.8 (DEF), U?.8 (VSS), U?.9 (GND), U?.9 (ST), U?.9 (VSS), X?.2 (GND), X?.4 (GND)
- new net M_CS: U?.4 (SPI_CS)
- new net USB_VBUS: J?.1 (VBUS), U?.2 (IN2)
- new net V_Bat: R?.2, U?.7 (IN1)
- new net V_bat: J?.1 (Pin_1)

Commit message: it didnt commite yesterday i dunno why
Parts:
- added C?: 10uF, symbol Device:C_Small
- added C?: 0.1uF, symbol Device:C_Small
- added C?: 10nF, symbol Device:C_Small
- added L?: 330nH, symbol Device:L_Small
- added R?: 100k, symbol Device:R_Small_US
Connections:
- net +3.3V: now also C?.2, C?.2, R?.2
- net GND: now also J?.1 (In), C?.1, C?.1, C?.1, L?.2
- net GPS_INT: now reaches U?.5 (EXTINT)
- net GPS_RST: now reaches U?.9 (RESET_N)
- net M_INT: now reaches U?.15 (INT)
- net at U?.21 (ANT): now also L?.1; no longer J?.1 (In)
- net TELE_RXM: now reaches U?.6 (RXEN)
- net TELE_TXM: now reaches U?.7 (TXEN)
- net STM32_RX renamed GPS_RX
- net STM32_TX renamed GPS_TX
- net TELE_RST: no longer names the net of U?.15 (NRST)
- net TELE_RST: now also C?.2, R?.1
Other:
- moved on the sheet: J?, U?
