File: S-Worm_PCB_Designs/S-Worm_PCB_Designs.kicad_sch (KiCad schematic)
At the start: 60 parts

Commit message: adc aaa
Parts:
- added R?: 30k, symbol Device:R_Small_US
- added R?: 7.5k, symbol Device:R_Small_US
Connections:
- net GND: now also R?.2
- net V_bat: now also R?.1
- new net V_sen: R?.1, R?.2
Other:
- moved on the sheet: C?, J?, R?, SW?, U?

Commit message: WHAT
Parts:
- added C31, C33: 0.1uF, symbol Device:C_Small
- added U9: ADS112U04IPWR, easyeda2kicad:TSSOP-16_L5.0-W4.4-P0.65-LS6.4-BL, symbol easyeda2kicad:ADS112U04IPWR
- gave numbers to parts that had none: 61
Connections:
- net IMU_CS is gone; now on net ICM_CS: U2.24 (PC4)
- net IMU_INT2 is gone; now on net ICM_INT2: U2.30 (PB11)
- net IMU_SCK is gone; now on net ICM_SCK: U2.21 (PA5)
- net IMU_SDI is gone; now on net ICM_SDI: U2.23 (PA7)
- net IMU_SDO is gone; now on net ICM_SDO: U2.22 (PA6)
- net TELE_MISO is gone; now on net TELE_SDO: U7.16 (MISO)
- net TELE_MOSI is gone; now on net TELE_SDI: U7.17 (MOSI)
- net TELE_NSS is gone; now on net TELE_CS: U7.19 (NSS)
- net V_bat is gone; now on net V_BAT: J4.1 (Pin_1), R5.1
- net +3.3V: now also C31.2, C33.1, U9.12 (AVDD), U9.13 (DVDD); no longer U3.4 (INT1/INT)
- net GND: now also C13.2, C9.2, J2.2 (Ext), U1.10 (GND), C31.1, C33.2, U9.4 (DGND), U9.5 (AVSS)
- net GPS_RX: now also U2.16 (PA2); no longer U2.17 (PA3)
- net GPS_TX: now also U2.17 (PA3); no longer U2.16 (PA2)
- net TELE_CS: no longer U2.27 (PB1)
- net V_RX: now reaches U2.14 (PA0-WKUP(PA0))
- net V_RX: now also U9.16 (RX)
- net V_TX: now reaches U2.15 (PA1)
- net V_TX: now also U9.15 (TX)
- net V_Bat renamed V_BAT
- new net ICM_INT1: U2.27 (PB1), U3.4 (INT1/INT)
- no-connect marks 5 -> 62
Other:
- moved on the sheet: C13, C16, C17, C18, C19, C22, C25, C26, C27, C28, C30, C32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

Commit message: yum
Parts:
- R6: value 7.5k -> 10k
Connections:
- net V_sen is gone; now on an unnamed net: R5.2, R6.1
- net GND: now also U1.12 (GND)
- no-connect marks 62 -> 60
Changed lines of the file:
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@@
 	)
 	(no_connect
-		(at 234.95 33.02)
-	)
-	(no_connect
 		(at 234.95 25.4)
 	)
@@
 	)
 	(no_connect
-		(at 72.39 137.16)
-	)
-	(no_connect
 		(at 100.33 45.72)
 	)
@@
 	(wire
 		(pts
+			(xy 233.68 33.02) (xy 234.95 33.02)
+		)
+		(stroke
+			(width 0)
+			(type default)
+		)
+	)
+	(wire
+		(pts
 			(xy 170.18 38.1) (xy 175.26 38.1)
 		)
@@
 	(wire
 		(pts
+			(xy 233.68 44.45) (xy 233.68 33.02)
+		)
+		(stroke
+			(width 0)
+			(type default)
+		)
+	)
+	(wire
+		(pts
 			(xy 173.99 85.09) (xy 173.99 90.17)
 		)
@@
 	(wire
 		(pts
+			(xy 204.47 33.02) (xy 204.47 44.45)
+		)
+		(stroke
+			(width 0)
+			(type default)
+		)
+	)
+	(wire
+		(pts
 			(xy 193.04 138.43) (xy 204.47 138.43)
 		)
@@
 	(wire
 		(pts
+			(xy 204.47 44.45) (xy 233.68 44.45)
+		)
+		(stroke
+			(width 0)
+			(type default)
+		)
+	)
+	(wire
+		(pts
 			(xy 148.59 142.24) (xy 148.59 144.78)
 		)
@@
 	(wire
 		(pts
-			(xy 208.28 33.02) (xy 200.66 33.02)
+			(xy 208.28 33.02) (xy 204.47 33.02)
 		)
 		(stroke
@@
 		)
 	)
-	(label "V_sen"
-		(at 200.66 33.02 0)
-		(effects
-			(font
-				(size 1.27 1.27)
-			)
-			(justify left bottom)
-		)
-	)
 	(label "USB_VBUS"
 		(at 166.37 54.61 0)
@@
 		(fields_autoplaced yes)
 		(property "Reference" "R6"
-			(at 213.995 35.56 90)
+			(at 210.82 34.2899 0)
 			(effects
 				(font
 					(size 1.27 1.27)
 				)
+				(justify left)
 			)
 		)
-		(property "Value" "7.5k"
-			(at 211.455 35.56 90)
+		(property "Value" "10k"
+			(at 210.82 36.8299 0)
 			(effects
 				(font
 					(size 1.27 1.27)
 				)
+				(justify left)
 			)
 		)
@@
 					(unit 1)
 				)
+			)
+		)
+	)
+	(symbol
+		(lib_id "power:GND")
+		(at 72.39 137.16 90)
+		(unit 1)
+		(exclude_from_sim no)
+		(in_bom yes)
+		(on_board yes)
+		(dnp no)
+		(fields_autoplaced yes)
+		(property "Reference" "#PWR050"
+			(at 78.74 137.16 0)
+			(effects
+				(font
+					(size 1.27 1.27)
+				)
+				(hide yes)
+			)
+		)
+		(property "Value" "GND"
+			(at 76.2 137.1599 90)
+			(effects
+				(font
+					(size 1.27 1.27)
+				)
+				(justify right)
+			)
+		)
+		(property "Footprint" ""
+			(at 72.39 137.16 0)
+			(effects
+				(font
+					(size 1.27 1.27)
+				)
+				(hide yes)
+			)
+		)
+		(property "Datasheet" ""
+			(at 72.39 137.16 0)
+			(effects
+				(font
+					(size 1.27 1.27)
+				)
+				(hide yes)
+			)
+		)
+		(property "Description" "Power symbol creates a global label with name \"GND\" , ground"
+			(at 72.39 137.16 0)
+			(effects
+				(font
+					(size 1.27 1.27)
+				)
+				(hide yes)
+			)
+		)
+		(pin "1"
+		)
+		(instances
+			(project ""
+				(path "/335fd408-0803-4c38-b9aa-8b4ba3fe733b"
+					(reference "#PWR050")
+					(unit 1)
+				)

Commit message: i dunno
Parts:
- removed FB1: FerriteBead_Small, symbol Device:FerriteBead_Small
- removed J4: Conn_01x02_Socket, symbol Connector:Conn_01x02_Socket
- added L1: FCM1608KF-601T03, easyeda2kicad:L0603, symbol easyeda2kicad:FCM1608KF-601T03
- added TP1: SP-_4, TestPoint:TestPoint_Pad_4.0x4.0mm, symbol Connector:TestPoint
- added TP10: 3.3v test pad, TestPoint:TestPoint_Pad_4.0x4.0mm, symbol Connector:TestPoint
- added TP11: GND test pad, TestPoint:TestPoint_Pad_4.0x4.0mm, symbol Connector:TestPoint
- added TP2: SP-_2, TestPoint:TestPoint_Pad_4.0x4.0mm, symbol Connector:TestPoint
- added TP3: SP-_3, TestPoint:TestPoint_Pad_4.0x4.0mm, symbol Connector:TestPoint
- added TP4: SP-_1, TestPoint:TestPoint_Pad_4.0x4.0mm, symbol Connector:TestPoint
- added TP5: SP+_4, TestPoint:TestPoint_Pad_4.0x4.0mm, symbol Connector:TestPoint
- added TP6: SP+_1, TestPoint:TestPoint_Pad_4.0x4.0mm, symbol Connector:TestPoint
- added TP7: SP+_3, TestPoint:TestPoint_Pad_4.0x4.0mm, symbol Connector:TestPoint
- added TP8: SP+_2, TestPoint:TestPoint_Pad_4.0x4.0mm, symbol Connector:TestPoint
- added TP9: Battery test pad, TestPoint:TestPoint_Pad_4.0x4.0mm, symbol Connector:TestPoint
- C1, C10, C11, C12, C13, C14, C15, C16, C17, C18, C2, C20, C21, C22, C23, C24, C25, C26, C28, C29, C3, C30, C31, C32, C33, C4, C6, C7, C8, C9: footprint (none) -> Capacitor_SMD:C_0402_1005Metric
- C19: footprint (none) -> Capacitor_SMD:C_0805_2012Metric
- C27, C5: value C -> 100nF; footprint (none) -> Capacitor_SMD:C_0402_1005Metric
- D1, D2, D3: footprint (none) -> LED_SMD:LED_0805_2012Metric
- J1: footprint (none) -> Connector_USB:USB_A_CNCTech_1001-011-01101_Horizontal
- J2, J3: footprint (none) -> Connector_Coaxial:U.FL_Hirose_U.FL-R-SMT-1_Vertical
- L2: renamed from L1; footprint (none) -> Inductor_SMD:L_0201_0603Metric
- L3: renamed from L2; footprint (none) -> Inductor_SMD:L_0201_0603Metric
- R1, R5, R6: footprint (none) -> Resistor_SMD:R_0201_0603Metric
- R2: renamed from R3; value R_Small_US -> 10k; footprint (none) -> Resistor_SMD:R_0201_0603Metric
- R3: renamed from R2; footprint (none) -> Resistor_SMD:R_0201_0603Metric
- R4, R7, R8: footprint (none) -> Resistor_SMD:R_0402_1005Metric
- renumbered SW2 to SW1, SW1 to SW2
Connections:
- net +3.3V: now also L1.1, TP10.1
- net GND: now also TP11.1, TP6.1
- net V_BAT: now also TP4.1, TP9.1
- net at U2.13 (VDDA): now also L1.2
- no-connect marks 60 -> 66
Other:
- moved on the sheet: R2, SW1

Commit message: almost there
Parts:
- removed L2: 330nH, Inductor_SMD:L_0201_0603Metric, symbol Device:L_Small
- added J4: Conn_01x03_Pin, Connector_JST:JST_ACH_BM03B-ACHSS-GAN-ETF_1x03-1MP_P1.20mm_Vertical, symbol Connector:Conn_01x03_Pin
- C1: value 10uF -> 4.7uF
- C2, C3, C4: value 1uF -> 4.7uF
- R3, R5, R6: footprint Resistor_SMD:R_0201_0603Metric -> Resistor_SMD:R_0402_1005Metric
- renumbered L3 to L2
Connections:
- net GND: now also J4.3 (Pin_3); no longer J3.1 (In)
- net V_BAT: now also J4.1 (Pin_1)
- net ESC_COM: now reaches U2.62 (PB9)
- net ESC_COM: now also J4.2 (Pin_2)
- net at U7.21 (ANT): now also J3.1 (In)
- no-connect marks 66 -> 65
